File: hw-module-gps.kicad_pcb (KiCad board)
At the start: 4 copper layers, 93.2 x 58 mm, 21 parts, among them J29 Conn_01x05, U12 AMS1117-3.3, U42 2.54mm 1x6 socket, U43 2.54mm 1x8 socket, U44 2.54mm 1x8 socket, U45 2.54mm 1x10 socket, U46 2.54mm 2x6 socket

Commit message: Initial Release
Parts:
- added kibuzzard-69B58D65: G***, kibuzzard-69B58D65, F.Cu at (236.4, 182.3)
- added kibuzzard-69B58D65: G***, kibuzzard-69B58D65, B.Cu at (232.2, 190.8)
- moved LOGO2 23.5 mm to (232.4, 140.5)
Connections:
- net /GPS/3.3V renamed /3.3V
- net /GPS/5V renamed /5V
- net /GPS/RXD renamed /RXD
- net /GPS/TXD renamed /TXD
Routing:
- net /TXD: track 48.1 -> 45.7 mm, vias 2 -> 1
Other:
- board text added: "5V"
- board text added: "GND"
- board text added: "N/C"
- board text added: "RXD"
- board text added: "TXD"

Commit message: updated CPL
Parts:
- removed U46: 2.54mm 2x6 socket, xtech:Dummy
