File: hw-module-gps.kicad_sch (KiCad schematic)
At the start: 19 parts, among them J29 Conn_01x05, U12 AMS1117-3.3, U42 2.54mm 1x6 socket, U43 2.54mm 1x8 socket, U44 2.54mm 1x8 socket, U45 2.54mm 1x10 socket, U46 2.54mm 2x6 socket

Commit message: updated CPL
Parts:
- removed U46: 2.54mm 2x6 socket, xtech:Dummy, symbol xtech:Dummy
